File: NEON_v2.11.sch (KiCad schematic (older format))
At the start: 29 parts, among them J1 B_1_SEL, J15 Conn_01x02, J2 USB_B_Micro, J24 B_0_SEL, J25 ST-LINK, SW1 SW_Push, U4 STM32F103RE, Y1 Crystal

Commit message: Updated MCU & Buck Library references
Parts:
- removed U4: STM32F103RE, Package_QFP:LQFP-64_10x10mm_P0.5mm, symbol Malloc_Library:STM32F103RE
- added U4: STM32F103RE, symbol mallocLibrarySCH:STM32F103RE
Connections:
- net +3V3: now also U4.13 (VDDA), U4.19 (VDD_4), U4.32 (VDD_1), U4.48 (VDD_2), U4.64 (VDD_3)
- net BOOT_0: now also U4.60 (BOOT0)
- net BOOT_1: now also U4.28 (PB2/BOOT1)
- net E_DIR: now also U4.10 (PC2/ADC123_IN12)
- net E_EN: now also U4.3 (PC14/OSC32_IN)
- net E_STEP: now also U4.4 (PC15/OSC32_OUT)
- net FAN_0: now also U4.26 (PB0/ADC12_IN8/TIM3_CH3/TIM8_CH2N/TIM1_CH2N)
- net FAN_1: now also U4.27 (PB1/ADC12_IN9/TIM3_CH4/TIM8_CH3N/TIM1_CH3N)
- net FAN_2: now also U4.14 (PA0/WKUP/USART2_CTS/ADC123_IN0/TIM2_CH1_ETR/TIM5_CH1/TIM8_ETR)
- net GND: now also U4.12 (VSSA), U4.18 (VSS_4), U4.31 (VSS_1), U4.47 (VSS_2), U4.63 (VSS_3)
- net Heatbed: now also U4.40 (PC9/TIM8_CH4/SDIO_D1/TIM3_CH4)
- net Hotend: now also U4.41 (PA8/USART1_CK/TIM1_CH1/MCO)
- net MISO_2: now also U4.22 (PA6/SPI1_MISO/ADC12_IN6/TIM3_CH1/TIM1_BKIN/TIM8_BKIN)
- net MOSI_2: now also U4.23 (PA7/SPI1_MOSI/ADC12_IN7/TIM3_CH2/TIM8_CH1N/TIM1_CH1N)
- net NRST: now also U4.7 (NRST)
- net PB10: now also U4.29 (PB10/I2C2_SCL/USART3_TX/TIM2_CH3)
- net PB11: now also U4.30 (PB11/I2C2_SDA/USART3_RX/TIM2_CH4)
- net PB12: now also U4.33 (PB12/SPI2_NSS/I2C2_SMBA/USART3_CK/TIM1_BKIN/I2S2_WS)
- net PB13: now also U4.34 (PB13/SPI2_SCK/I2S2_CK/USART3_CTS/TIM1_CH1N)
- net SCK_2: now also U4.21 (PA5/SPI1_SCK/ADC12_IN5/DAC_OUT2)
- net SCL: now also U4.58 (PB6/I2C1_SCL/TIM4_CH1/USART1_TX)
- net SDA: now also U4.59 (PB7/I2C1_SDA/TIM4_CH2/USART1_RX)
- net SDCS: now also U4.25 (PC5/ADC12_IN15)
- net STM_RX_1: now also U4.43 (PA10/USART1_RX/TIM1_CH3)
- net STM_RX_2: now also U4.17 (PA3/USART2_RX/ADC123_IN3/TIM2_CH4/TIM5_CH4)
- net STM_RX_4: now also U4.52 (PC11/UART4_RX/SDIO_D3/USART3_RX)
- net STM_TX_1: now also U4.42 (PA9/USART1_TX/TIM1_CH2)
- net STM_TX_2: now also U4.16 (PA2/USART2_TX/ADC123_IN2/TIM2_CH3/TIM5_CH3)
- net STM_TX_4: now also U4.51 (PC10/UART4_TX/SDIO_D2/USART3_TX)
- net SWDCLK: now also U4.49 (JTCK/SWCLK/PA14)
- net SWDIO: now also U4.46 (JTMS/SWDIO/PA13)
- net Servo_0: now also U4.50 (JTDI/SPI3_NSS/I2S3_WS/TIM2_CH1_ETR/PA15/SPI1_NSS)
- net Servo_1: now also U4.54 (PD2/TIM3_ETR/UART5_RX/SDIO_CMD)
- net Temp_0: now also U4.24 (PC4/ADC12_IN14)
- net Temp_1: now also U4.20 (PA4/SPI1_NSS/USART2_CK/ADC12_IN4/DAC_OUT1)
- net USB+: now also U4.45 (PA12/USART1_RTS/CANTX/USBDP/TIM1_ETR)
- net USB-: now also U4.44 (PA11/USART1_CTS/CANRX/USBDM/TIM1_CH4)
- net X_DIR: now also U4.38 (PC7/I2S3_MCK/TIM8_CH2/SDIO_D7/TIM3_CH2)
- net X_EN: now also U4.53 (PC12/UART5_TX/SDIO_CK/USART3_CK)
- net X_Min: now also U4.35 (PB14/SPI2_MISO/USART3_RTS/TIM1_CH2N)
- net X_STEP: now also U4.39 (PC8/TIM8_CH3/SDIO_D0/TIM3_CH3)
- net Y_DIR: now also U4.57 (PB5/I2C1_SMBA/SPI3_MOSI/I2S3_SD/TIM3_CH2/SPI1_MOSI)
- net Y_EN: now also U4.55 (JTDO/SPI3_SCK/I2S3_CK/TIM2_CH2/PB3/TRACESWO/SPI1_SCK)
- net Y_Min: now also U4.36 (PB15/SPI2_MOSI/TIM1_CH3N/I2S2_SD)
- net Y_STEP: now also U4.56 (JNTRST/SPI3_MISO/TIM3_CH1/PB4/SPI1_MISO)
- net Z_2_DIR: now also U4.2 (PC13/TMPR/RTC)
- net Z_2_EN: now also U4.9 (PC1/ADC123_IN11)
- net Z_2_STEP: now also U4.8 (PC0/ADC123_IN10)
- net Z_DIR: now also U4.15 (PA1/USART2_RTS/ADC123_IN1/TIM2_CH2/TIM5_CH2)
- net Z_EN: now also U4.61 (PB8/TIM4_CH3/SDIO_D4/I2C1_SCL/CANRX)
- net Z_Min: now also U4.37 (PC6/I2S2_MCK/TIM8_CH1/SDIO_D6/TIM3_CH1)
- net Z_STEP: now also U4.62 (PB9/TIM4_CH4/SDIO_D5//I2C1_SDA/CANTX)
- net at C18.1, Y1.1: now also U4.5 (OSC_IN/PD0/CANRX)
- net at C19.1, Y1.2: now also U4.6 (OSC_OUT/PD1/CANTX)
Changed lines of the file:
@@
 	2700 3200 2600 3200
-Wire Wire Line
-	2600 3200 2600 3900
 Wire Wire Line
 	2700 3900 2600 3900
@@
 PB11
 $Comp
-L Malloc_Library:STM32F103RE U?
-U 1 1 5D364B10
-P 5900 1600
-AR Path="/5D362114/5D364B10" Ref="U?"  Part="1"
-AR Path="/5D364B10" Ref="U4"  Part="1"
-F 0 "U4" H 5900 1765 50  0000 C CNN
-F 1 "STM32F103RE" H 5900 1674 50  0000 C CNN
-F 2 "Package_QFP:LQFP-64_10x10mm_P0.5mm" H 5800 1600 50  0001 C CNN
-F 3 "" H 5800 1600 50  0001 C CNN
-F 4 " C8322" H 5900 1600 50  0001 C CNN "JLC"
-	1    5900 1600
-	1    0    0    -1
-$EndComp
-$Comp
 L Device:C C?
 U 1 1 5E085891
@@
 Text GLabel 1100 6500 0    50   Input ~ 0
 NRST
+Wire Wire Line
+	2600 3200 2600 3900
+$Comp
+L mallocLibrarySCH:STM32F103RE U4
+U 1 1 5EF7AF69
+P 5900 1600
+F 0 "U4" H 5900 1765 50  0000 C CNN
+F 1 "STM32F103RE" H 5900 1674 50  0000 C CNN
+F 2 "" H 5800 1600 50  0001 C CNN
+F 3 "" H 5800 1600 50  0001 C CNN
+	1    5900 1600
+	1    0    0    -1
+$EndComp
 $EndSCHEMATC
