File: Power.sch (KiCad schematic (older format))
At the start: 30 parts, among them J13 +12V_IN, J14 V_Heatbed_IN, J21 Conn_02x06_Odd_Even, U1 TPS5430, U2 AP1117-33

Commit message: Updated MCU & Buck Library references
Parts:
- U1: symbol Malloc_Library:TPS5430 -> mallocLibrarySCH:TPS5430
Changed lines of the file:
@@
 $EndComp
 $Comp
-L Malloc_Library:TPS5430 U1
+L mallocLibrarySCH:TPS5430 U1
 U 1 1 5D859A5C
 P 5800 2150
